Commit message: M5: end-to-end scenarios and launch tests, camera noise switch, auto GPU default
Scenario files E1-E12, a parametrised launch_testing harness scored against ground truth,
camera_noise argument for E11, gpu:=auto default (NVIDIA when usable), box_a moved so
marker 0 is visible from the marker 4 dock (E12), E7 spawn settled.

File: src/dockbot_description/urdf/dockbot.urdf.xacro (robot description, xacro)
@@ -13,4 +13,7 @@
   <xacro:arg name="camera_fov" default="1.0856"/>
   <xacro:arg name="camera_rate" default="30"/>
+  <!-- Standard deviation of Gaussian pixel noise (0 to 1 of full scale); 0 turns the noise off. -->
+  <xacro:arg name="camera_noise" default="0.0"/>
+  <xacro:property name="camera_noise" value="$(arg camera_noise)"/>
   <xacro:property name="chassis_l" value="0.30"/>
   <xacro:property name="chassis_w" value="0.24"/>
@@ -212,4 +215,11 @@
         </image>
         <clip><near>0.05</near><far>20.0</far></clip>
+        <xacro:if value="${camera_noise &gt; 0.0}">
+          <noise>
+            <type>gaussian</type>
+            <mean>0.0</mean>
+            <stddev>${camera_noise}</stddev>
+          </noise>
+        </xacro:if>
       </camera>
     </sensor>
